File: J-ST-Link.sch (EAGLE design)
At the start: 17 parts, among them IC1 TLV70433, J5 SOLDERJUMPER_2WAY_CLOSED, J7 SOLDERJUMPER_2WAY_CLOSED, J9 SOLDERJUMPER_2WAY_CLOSED

Commit message: Optimised schematic
Parts:
- R1: value 1K -> 330R
Connections:
- net SWIM_RST renamed !SWIM_RST
- net VTREF renamed VCC
Other:
- moved on the sheet: 10-127, J5, J7, J9
